File: kicad7.0_files/D1-mini-macro/D1-mini-macro.kicad_pcb (KiCad board)
At the start: 2 copper layers, 45 x 96.1 mm, 9 parts

Commit message: update to rear silk screen
updated rear silk screen to show voltage in for 5v and 3.3v and updated screen shot
Parts:
- renumbered REF** to wemos-D1-mini
Other:
- board text added: "3V3 IN - +"
- board text added: "5V IN - +"
Changed lines of the file:
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@@
     (at 148.088051 160.6542)
     (attr through_hole)
-    (fp_text reference "REF**" (at -0.9318 0.381 90 unlocked) (layer "F.SilkS")
+    (fp_text reference "wemos-D1-mini" (at -0.9318 0.381 90 unlocked) (layer "F.SilkS")
         (effects (font (size 1 1) (thickness 0.1)))
     )
-    (fp_text value "wemos-D1-mini" (at 0.5682 0.381 90 unlocked) (layer "F.Fab")
+    (fp_text value "wemos-D1-mini" (at 0.5682 0.381 90 unlocked) (layer "F.Fab") hide
         (effects (font (size 1 1) (thickness 0.15)))
     )
@@
         (effects (font (size 1 1) (thickness 0.1)) (justify left bottom))
     )
-    (fp_text user "${REFERENCE}" (at 2.0682 0.381 90 unlocked) (layer "F.Fab")
+    (fp_text user "${REFERENCE}" (at 2.0682 0.381 90 unlocked) (layer "F.Fab") hide
         (effects (font (size 1 1) (thickness 0.15)))
     )
@@
   (gr_arc (start 169.53455 179.675899) (mid 168.649251 181.8132) (end 166.51195 182.698499)
     (stroke (width 0.1) (type default)) (layer "Edge.Cuts"))
+  (gr_text "3V3 IN\n-    +" (at 142.6718 139.2174) (layer "B.SilkS")
+    (effects (font (size 1 1) (thickness 0.125)) (justify left bottom mirror))
+  )
+  (gr_text "5V  IN\n-    +" (at 157.8102 139.3698) (layer "B.SilkS")
+    (effects (font (size 1 1) (thickness 0.125)) (justify left bottom mirror))
+  )
   (gr_text "-" (at 147.516451 137.2616) (layer "F.SilkS")
     (effects (font (size 1 1) (thickness 0.125)) (justify left bottom))

Commit message: added resister for LED
updated PCB files and png
Parts:
- added ?: , , F.Cu at (128.0, 170.7)
- added R1 for LED: R_Axial_DIN0204_L3.6mm_D1.6mm_P5.08mm_Horizontal, Resistor_THT:R_Axial_DIN0204_L3.6mm_D1.6mm_P5.08mm_Horizontal, F.Cu at (132.2, 172.3)
- added R=0: SolderWirePad_1x01_SMD_1x2mm, Connector_Wire:SolderWirePad_1x01_SMD_1x2mm, F.Cu at (128.0, 169.1)
- added The Handsome Zebra: LOGO, LOGO, B.Cu at (147.2, 114.0)
Routing:
- net (no net): track 507.3 -> 520.7 mm
Other:
- board text added: "The Handsome Zebra"
